File: dcdc.kicad_pcb (KiCad board)
At the start: 4 copper layers, 58 x 59 mm, 122 parts, among them J1 Conn_01x04_Pin, J2 Conn_01x04_Pin, Q1 IPD025N06N, Q2 IPD025N06N, SW1 SW_Omron_B3FS, SW2 SW_Omron_B3FS, SW3 SW_Omron_B3FS, U1 LP5907MFX-3.3, U2 LM5164DDA, U3 LM5164DDA, U4 INA282, U5 UCC27201A, U6 OPA2333xxD, U7 STM32F334C8Tx, Y1 CSTCE12M

Commit message: 完成
Parts:
- removed the R29 at (168.8, 74.5)
- added C24: 100n, Capacitor_SMD:C_0603_1608Metric, B.Cu at (150.8, 128.8)
- added C28: 100n, Capacitor_SMD:C_0603_1608Metric, B.Cu at (166.3, 114.3)
- added R33: 10k, Resistor_SMD:R_0603_1608Metric, F.Cu at (168.8, 74.5)
- L3: value 47u -> 68u
- R14: value 2m -> 20m; moved to B.Cu
- R24: value R -> 33
- R28, R34: value 100 -> 10k
- R35, R36: value 1k -> 10k
- U4: value INA282 -> INA240A1PW; footprint Package_SO:SOIC-8_3.9x4.9mm_P1.27mm -> Package_SO:TSSOP-8_4.4x3mm_P0.65mm
- moved U4 25.3 mm to (145.8, 128.7), turned to 0 degrees
- moved R14 20.9 mm to (142.8, 124.5), turned to 0 degrees
- moved L3 0.25 mm to (133.1, 124.9)
- moved R28 0.08 mm to (147.8, 74.5), turned to 0 degrees
- moved R34 0.05 mm to (158.1, 74.5), turned to 0 degrees
- renumbered C24 to C25, C25 to C26, C26 to C27, C27 to C29, C28 to C30, C29 to C31, C30 to C32, C31 to C33, C32 to C34, C33 to C35, C34 to C36, C35 to C37, C36 to C38, C37 to C39, C38 to C40, C39 to C41, C40 to C42, C41 to C43, C42 to C44, C43 to C45, C44 to C46, C45 to C47, C46 to C48, D12 to D10, D13 to D11, D14 to D12, D15 to D13, D16 to D14, D17 to D15, D18 to D16, D19 to D17, D10 to D8, D11 to D9, VIN to H1, GND to H2, VOUT to H3, GND to H4, R30 to R29, R31 to R30, R32 to R31, R33 to R32, RESET to SW4
Connections:
- C27 pad 1: VC -> I-
- C29 pad 1: VC -> I-
- C31 pad 1: VC -> I-
- C33 pad 1: VC -> I-
- C34 pad 2: I+ -> SW
- C35 pad 1: VC -> I-
- C38 pad 1: Net-(C36-Pad1) -> PB7
- C39 pad 1: Net-(C37-Pad1) -> PB5
- C40 pad 1: Net-(C38-Pad1) -> PB6
- D12 pad 1: VC -> I-
- D4 pad 2: I+ -> SW
- H3 pad 1: VC -> I-
- L3 pad 1: I- -> SW
- L3 pad 2: VC -> I+
- Q1 pad 3: I+ -> SW
- Q2 pad 2: I+ -> SW
- R27 pad 2: VC -> I-
- R28 pad 1: Net-(C36-Pad1) -> +3V3
- R34 pad 1: Net-(C38-Pad1) -> +3V3
- R9 pad 2: I+ -> SW
- U4 pad 1: I- -> GND
- U4 pad 2: GND -> I+
- U4 pad 3: +3V3 -> I-
- U4 pad 4: unconnected-(U4-NC-Pad4) -> GND
- U4 pad 5: Net-(R22-Pad2) -> +3V3
- U4 pad 8: I+ -> Net-(R22-Pad2)
- U5 pad 4: I+ -> SW
Routing:
- net +3V3: track 180.8 -> 253.1 mm, vias 9 -> 11
- net Net-(R22-Pad2): track 28.5 -> 71.1 mm
- net SW: track 0.00 -> 9.39 mm, vias 0 -> 16
- net VC: track 8.29 -> 0.00 mm, vias 33 -> 0
- net I+: track 12.3 -> 6.99 mm, vias 2 -> 3
- net PB7: track 24.0 -> 29.3 mm
- net PB5: track 43.8 -> 49.0 mm
- net PB6: track 33.4 -> 38.3 mm
- net I-: track 1.82 -> 5.94 mm, vias 1 -> 14
- net Net-(C38-Pad1): track 1.65 -> 0.00 mm
- net Net-(C36-Pad1): track 1.65 -> 0.00 mm
- net Net-(C37-Pad1): track 1.62 -> 0.00 mm
- net GND: track 78.2 -> 79.5 mm, vias 68 -> 73
- added copper zone on B.Cu, net I-
- added copper zone on B.Cu, net SW
- added copper zone on F.Cu, net SW
- removed copper zone on F.Cu, net I+
- removed copper zone on B.Cu, net VC
- removed copper zone on F.Cu, net VC
Other:
- board size 58 x 59 mm -> 58 x 59.2 mm
