File: dcdc.kicad_sch (KiCad schematic)
At the start: 122 parts, among them J1 Conn_01x04_Pin, J2 Conn_01x04_Pin, Q1 IPD025N06N, Q2 IPD025N06N, SW1 SW_Omron_B3FS, SW2 SW_Omron_B3FS, SW3 SW_Omron_B3FS, SW4 SW_Omron_B3FS, U1 LP5907MFX-3.3, U2 LM5164DDA, U3 LM5164DDA, U4 INA282, U5 UCC27201A, U6 OPA2333xxD, U7 STM32F334C8Tx, Y1 CSTCE12M

Commit message: 完成
Parts:
- removed R29: 100, Resistor_SMD:R_0603_1608Metric, symbol Device:R
- removed U4: INA282, Package_SO:SOIC-8_3.9x4.9mm_P1.27mm, symbol Amplifier_Current:INA282
- added C24, C28: 100n, Capacitor_SMD:C_0603_1608Metric, symbol Device:C_Small
- added R33: 10k, Resistor_SMD:R_0603_1608Metric, symbol Device:R
- added U4: INA240A1PW, Package_SO:TSSOP-8_4.4x3mm_P0.65mm, symbol Amplifier_Current:INA240A1PW
- R14: value 2m -> 20m
- R28, R34: value 100 -> 10k
- R35, R36: value 1k -> 10k
- renumbered C24 to C25, C25 to C26, C26 to C27, C27 to C29, C28 to C30, C29 to C31, C30 to C32, C31 to C33, C32 to C34, C33 to C35, C34 to C36, C35 to C37, C36 to C38, C37 to C39, C38 to C40, C39 to C41, C40 to C42, C41 to C43, C42 to C44, C43 to C45, C44 to C46, C45 to C47, C46 to C48, D12 to D10, D13 to D11, D14 to D12, D15 to D13, D16 to D14, D17 to D15, D18 to D16, D19 to D17, D10 to D8, D11 to D9, R30 to R29, R31 to R30, R32 to R31, R33 to R32
Connections:
- net +3V3: now also R28.1, R34.1, C24.1, C28.1, R33.1, U4.5 (V+), U4.6 (REF2)
- net GND: now also C24.2, C28.2, U4.1 (GND), U4.4 (GND), U4.7 (REF1)
- net I+: now also L3.2, U4.2 (+); no longer C34.2, D4.2 (A2), Q1.3 (S), Q2.2 (D), R9.2, U5.4 (HS)
- net I-: now also C27.1, C29.1, C31.1, C33.1, C35.1, D12.1 (K), H3.1, R27.2, U4.3 (-); no longer L3.1
- net PB5: now also C39.1, R33.2
- net PB6: now also C40.1
- net PB7: now also C38.1
- net at R22.2: now also U4.8
- removed net VC: C27.1, C29.1, C31.1, C33.1, C35.1, D12.1 (K), H3.1, L3.2, R27.2
- new net SW: C34.2, D4.2 (A2), L3.1, Q1.3 (S), Q2.2 (D), R9.2, U5.4 (HS)
Other:
- moved on the sheet: C32, D9, L3, R14, R22
